File: PYNQ/KiCad Schematics/Rx/Rx.kicad_sch (KiCad schematic)
At the start: 4 parts

Commit message: updated Rx pynq kiCad schematic
Parts:
- removed Grover1: ~, symbol CapstoneSymbols:Grover
- added Grover Shield1: ~, symbol CapstoneSymbols:Grover Shield
Connections:
- net at R1.1, Ultrasonic Piezoelectric Transducer1. (Red): now also Grover Shield1. (VCC)
- net at R1.2, Ultrasonic Piezoelectric Transducer1. (Red): now also Grover Shield1. (VCC)
Other:
- moved on the sheet: PYNQ1, R1, Ultrasonic Piezoelectric Transducer1
Changed lines of the file:
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@@
 	(paper "A4")
 	(junction
-		(at 187.96 34.29)
+		(at 114.3 38.1)
 		(diameter 0)
 		(color 0 0 0 0)
 	)
 	(junction
-		(at 187.96 41.91)
+		(at 114.3 45.72)
 		(diameter 0)
 		(color 0 0 0 0)
@@
 	(wire
 		(pts
-			(xy 200.66 36.83) (xy 200.66 34.29)
-		)
-		(stroke
-			(width 0)
-			(type default)
-		)
-	)
-	(wire
-		(pts
-			(xy 168.91 41.91) (xy 187.96 41.91)
-		)
-		(stroke
-			(width 0)
-			(type default)
-		)
-	)
-	(wire
-		(pts
-			(xy 187.96 41.91) (xy 200.66 41.91)
-		)
-		(stroke
-			(width 0)
-			(type default)
-		)
-	)
-	(wire
-		(pts
-			(xy 200.66 39.37) (xy 200.66 41.91)
-		)
-		(stroke
-			(width 0)
-			(type default)
-		)
-	)
-	(wire
-		(pts
-			(xy 200.66 34.29) (xy 187.96 34.29)
-		)
-		(stroke
-			(width 0)
-			(type default)
-		)
-	)
-	(wire
-		(pts
-			(xy 187.96 34.29) (xy 168.91 34.29)
+			(xy 127 40.64) (xy 127 38.1)
+		)
+		(stroke
+			(width 0)
+			(type default)
+		)
+	)
+	(wire
+		(pts
+			(xy 114.3 45.72) (xy 127 45.72)
+		)
+		(stroke
+			(width 0)
+			(type default)
+		)
+	)
+	(wire
+		(pts
+			(xy 127 43.18) (xy 127 45.72)
+		)
+		(stroke
+			(width 0)
+			(type default)
+		)
+	)
+	(wire
+		(pts
+			(xy 127 38.1) (xy 114.3 38.1)
+		)
+		(stroke
+			(width 0)
+			(type default)
+		)
+	)
+	(wire
+		(pts
+			(xy 101.6 38.1) (xy 114.3 38.1)
+		)
+		(stroke
+			(width 0)
+			(type default)
+		)
+	)
+	(wire
+		(pts
+			(xy 101.6 45.72) (xy 114.3 45.72)
 		)
 		(stroke
@@
 	(text "Rx"
 		(exclude_from_sim no)
-		(at 199.898 65.278 0)
+		(at 132.588 69.088 0)
 		(effects
 			(font
@@
 	(symbol
 		(lib_id "Device:R")
-		(at 187.96 38.1 0)
+		(at 114.3 41.91 0)
 		(unit 1)
 		(exclude_from_sim no)
@@
 		(fields_autoplaced yes)
 		(property "Reference" "R1"
-			(at 190.5 36.8299 0)
+			(at 116.84 40.6399 0)
 			(effects
 				(font
@@
 		)
 		(property "Value" "10 ohms"
-			(at 190.5 39.3699 0)
+			(at 116.84 43.1799 0)
 			(effects
 				(font
@@
 		)
 		(property "Footprint" ""
-			(at 186.182 38.1 90)
+			(at 112.522 41.91 90)
 			(effects
 				(font
@@
 		)
 		(property "Datasheet" "~"
-			(at 187.96 38.1 0)
+			(at 114.3 41.91 0)
 			(effects
 				(font
@@
 		)
 		(property "Description" "Resistor"
-			(at 187.96 38.1 0)
+			(at 114.3 41.91 0)
 			(effects
 				(font
@@
 	(symbol
 		(lib_id "CapstoneSymbols:Ultrasonic_Piezoelectric_Transducer")
-		(at 207.01 33.02 0)
+		(at 133.35 36.83 0)
 		(unit 1)
 		(exclude_from_sim no)
@@
 		(fields_autoplaced yes)
 		(property "Reference" "Ultrasonic Piezoelectric Transducer1"
-			(at 212.09 37.4649 0)
+			(at 138.43 41.2749 0)
 			(effects
 				(font
@@
 		)
 		(property "Value" "~"
-			(at 212.09 39.37 0)
+			(at 138.43 43.18 0)
 			(effects
 				(font
@@
 		)
 		(property "Footprint" ""
-			(at 207.01 33.02 0)
+			(at 133.35 36.83 0)
 			(effects
 				(font
@@
 		)
 		(property "Datasheet" ""
-			(at 207.01 33.02 0)
+			(at 133.35 36.83 0)
 			(effects
 				(font
@@
 		)
 		(property "Description" ""
-			(at 207.01 33.02 0)
+			(at 133.35 36.83 0)
 			(effects
 				(font
@@
 	)
 	(symbol
-		(lib_id "CapstoneSymbols:Grover")
-		(at 137.16 68.58 90)
-		(unit 1)
-		(exclude_from_sim no)
-		(in_bom yes)
-		(on_board yes)
-		(dnp no)
-		(fields_autoplaced yes)
-		(property "Reference" "Grover1"
-			(at 150.495 19.05 90)
-			(effects
-				(font
-					(size 2.54 2.54)
-				)
-			)
-		)
-		(property "Value" "~"
-			(at 150.495 22.86 90)
-			(effects
-				(font
-					(size 1.27 1.27)
-				)
-			)
-		)
-		(property "Footprint" ""
-			(at 137.16 68.58 0)
-			(effects
-				(font
-					(size 1.27 1.27)
-				)
-				(hide yes)
-			)
-		)
-		(property "Datasheet" ""
-			(at 137.16 68.58 0)
-			(effects
-				(font
-					(size 1.27 1.27)
-				)
-				(hide yes)
-			)
-		)
-		(property "Description" ""
-			(at 137.16 68.58 0)
-			(effects
-				(font
-					(size 1.27 1.27)
-				)
-				(hide yes)
-			)
-		)
-		(pin ""
-		)
-		(pin ""
-		)
-		(pin ""
-		)
-		(pin ""
-		)
-		(pin ""
-		)
-		(pin ""
-		)
-		(pin ""
-		)
-		(pin ""
-		)
-		(pin ""
-		)
-		(pin ""
-		)
-		(pin ""
-		)
-		(pin ""
-		)
-		(pin ""
-		)
-		(pin ""
-		)
-		(pin ""
-		)
-		(pin ""
-		)
-		(instances
-			(project "Rx"
-				(path "/5bfd56d5-c28e-473d-8c6f-8780ca293668"
-					(reference "Grover1")
-					(unit 1)
-				)
-			)
-		)
-	)
-	(symbol
 		(lib_id "CapstoneSymbols:PYNQ-Z2")
 		(at 63.5 69.85 0)
+		(mirror y)
 		(unit 1)
 		(exclude_from_sim no)
@@
 		(dnp no)
 		(property "Reference" "PYNQ1"
-			(at 62.992 25.4 0)
+			(at 38.1 32.766 0)
 			(effects
 				(font
@@
 		)
 		(property "Value" "~"
-			(at 64.135 19.05 0)
+			(at 62.865 19.05 0)
 			(effects
 				(font
@@
 					(unit 1)
 				)
+			)
+		)
+	)
+	(symbol
+		(lib_id "CapstoneSymbols:Grover Shield")
+		(at 69.85 72.39 90)
+		(unit 1)
+		(exclude_from_sim no)
+		(in_bom yes)
+		(on_board yes)
+		(dnp no)
+		(property "Reference" "Grover Shield1"
+			(at 76.454 32.512 90)
+			(effects
+				(font
+					(size 2.54 2.54)
+				)
+			)
+		)
+		(property "Value" "~"
+			(at 83.185 26.67 90)
+			(effects
+				(font
+					(size 1.27 1.27)
+				)
+			)
+		)
+		(property "Footprint" ""
+			(at 69.85 72.39 0)
+			(effects
+				(font
+					(size 1.27 1.27)
+				)
+				(hide yes)
+			)
+		)
+		(property "Datasheet" ""
+			(at 69.85 72.39 0)
+			(effects
+				(font
+					(size 1.27 1.27)
+				)
+				(hide yes)
+			)
+		)
+		(property "Description" ""
+			(at 69.85 72.39 0)
+			(effects
+				(font
+					(size 1.27 1.27)
+				)
+				(hide yes)
+			)
+		)
+		(pin ""
+		)
+		(pin ""
+		)
+		(pin ""
+		)
+		(pin ""
+		)
+		(pin ""
+		)
+		(pin ""
+		)
+		(pin ""
+		)
+		(pin ""
+		)
+		(pin ""
+		)
+		(pin ""
+		)
+		(pin ""
+		)
+		(pin ""
+		)
+		(pin ""
+		)
+		(pin ""
+		)
+		(pin ""
+		)
+		(pin ""
+		)
+		(instances
+			(project "Rx"
+				(path "/5bfd56d5-c28e-473d-8c6f-8780ca293668"
+					(reference "Grover Shield1")
+					(unit 1)
+				)
